Commit message: 04/21 urdf_xacro セッティング

File: urdf/old/arno.urdf (robot description, URDF)
Before this commit: robot icart_mini, 11 links, 10 joints
Joints:
- joint laser_joint1: origin xyz=0 0.25 0.670 rpy=3.141592653589793 0 1.3 -> xyz=0.2 0.0 0.30 rpy=0 0 0
- joint laser_joint2: origin xyz=0 -0.25 0.67 rpy=3.141592653589793 0 -1.3 -> xyz=-0.3 0.0 0.30 rpy=0 0 3.141592653589793
- joint laser_joint4: origin xyz=0.25 0 0.3 rpy=0 0 0 -> xyz=0.15 0 0.3 rpy=0 0 0

File: urdf/old/arno.xacro (robot description, xacro)
@@ -121,5 +121,5 @@
     <parent link="base_link"/>
     <child  link="ust"/>
-    <origin xyz="0 0.25 0.670" rpy="3.141592653589793 0 1.3"/>
+    <origin xyz="0.2 0.0 0.30" rpy="0 0 0"/>
   </joint>
   <link name="ust">
@@ -141,5 +141,5 @@
     <parent link="base_link"/>
     <child  link="ust2"/>
-    <origin xyz="0 -0.25 0.67" rpy="3.141592653589793 0 -1.3"/>
+    <origin xyz="-0.3 0.0 0.30" rpy="0 0 ${PI}"/>
   </joint>
   <link name="ust2">
@@ -181,5 +181,5 @@
     <parent link="base_link"/>
     <child  link="ylm"/>
-    <origin rpy="0 0 0" xyz="0.25 0 0.3"/>
+    <origin xyz="0.15 0 0.3" rpy="0 0 0"/>
   </joint>
   <link name="ylm">
