Commit message: nara2

File: urdf/arno.urdf (robot description, URDF)
Before this commit: robot icart_mini, 11 links, 10 joints
Links:
- link base_link: mass 20 -> None

File: urdf/arno.xacro (robot description, xacro)
@@ -34,9 +34,10 @@
       </geometry>
     </visual>
+    <!--
     <inertial>
        <mass value="20" />
        <origin xyz="-0.08 0 0" rpy="0 0 0"/>
        <inertia ixx="1" ixy="0" ixz="0" iyy="1" iyz="0" izz="1" />
-    </inertial>
+    </inertial> -->
   </link>
   <link name="left_wheel">
